File: syth_mcu/dac-pchannel.kicad_sch (KiCad schematic)
At the start: 23 parts, among them J4 AudioPlug3, Q1 SI2307DS, Q2 SI2304DS, Q3 SI2307DS, Q4 SI2304DS

Commit message: update layout
Parts:
- C1: value 80nF -> 100nF
- C5, C7: footprint Capacitor_THT:C_Rect_L9.0mm_W3.2mm_P7.50mm_MKT -> Capacitor_THT:CP_Radial_D5.0mm_P2.00mm
Changed lines of the file:
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@@
 			)
 		)
-		(property "Value" "80nF"
+		(property "Value" "100nF"
 			(at 77.47 67.3099 0)
 			(show_name no)
@@
 			)
 		)
-		(property "Footprint" "Capacitor_THT:C_Rect_L9.0mm_W3.2mm_P7.50mm_MKT"
+		(property "Footprint" "Capacitor_THT:CP_Radial_D5.0mm_P2.00mm"
 			(at 105.1052 102.87 0)
 			(hide yes)
@@
 			)
 		)
-		(property "Footprint" "Capacitor_THT:C_Rect_L9.0mm_W3.2mm_P7.50mm_MKT"
+		(property "Footprint" "Capacitor_THT:CP_Radial_D5.0mm_P2.00mm"
 			(at 105.1052 46.99 0)
 			(hide yes)
