File: syth_mcu/dac-pchannel.kicad_sch (KiCad schematic)
At the start: 23 parts, among them J3 PJ-320A, Q1 SI2307DS, Q2 SI2304DS, Q3 SI2307DS, Q4 SI2304DS

Commit message: schematic v2: LED indicator, RV6-8 pots, CHAIN GPIO labels (PC14/PC15); renumber RV refs in dac-pchannel
Parts:
- renumbered RV6 to RV13, RV7 to RV14
Changed lines of the file:
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@@
 		(in_pos_files yes)
 		(dnp no)
-		(property "Reference" "RV6"
+		(property "Reference" "RV13"
 			(at 101.6 73.6601 0)
 			(show_name no)
@@
 			(project "syth_mcu"
 				(path "/6f6073ad-48fd-4b64-b32f-c8e9bfc21ddc/de801ae6-5eb3-45eb-b018-1b4139932f15"
-					(reference "RV6")
+					(reference "RV13")
 					(unit 1)
 				)
@@
 		(in_pos_files yes)
 		(dnp no)
-		(property "Reference" "RV7"
+		(property "Reference" "RV14"
 			(at 101.6 128.2701 0)
 			(show_name no)
@@
 			(project "syth_mcu"
 				(path "/6f6073ad-48fd-4b64-b32f-c8e9bfc21ddc/de801ae6-5eb3-45eb-b018-1b4139932f15"
-					(reference "RV7")
-					(unit 1)
-				)
+					(reference "RV14")
+					(unit 1)
+				)
