File: syth_mcu/syth_mcu.kicad_sch (KiCad schematic)
At the start: 32 parts, among them J1 Conn_01x05, J2 Conn_01x05, J3 USB_C_Receptacle_PowerOnly_6P, J5 Conn_01x20, J6 Conn_01x20, J7 Conn_01x16, J8 Conn_01x08, J9 Conn_01x07, SW1 SW_Push, SW2 SW_Push, SW3 SW_Push, SW4 SW_Push, SW5 SW_Push, U2 YAAJ_WeAct_BlackPill_Part_Like, U3 AMS1117-3.3, U4 AMS1117-3.3, U5 TFT_320x240

Commit message: update layout
Parts:
- U5: footprint Connector_PinHeader_2.54mm:PinHeader_1x14_P2.54mm_Vertical -> Connector_PinSocket_2.54mm:PinSocket_1x14_P2.54mm_Vertical
Changed lines of the file:
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@@
 			)
 		)
-		(property "Footprint" "Connector_PinHeader_2.54mm:PinHeader_1x14_P2.54mm_Vertical"
+		(property "Footprint" "Connector_PinSocket_2.54mm:PinSocket_1x14_P2.54mm_Vertical"
 			(at 214.63 123.1899 0)
 			(show_name no)

Commit message: update layout
Parts:
- added J10, J11: Conn_01x20, Connector_PinSocket_2.54mm:PinSocket_1x20_P2.54mm_Vertical, symbol Connector_Generic:Conn_01x20
- J5, J6: footprint Connector_PinSocket_2.54mm:PinSocket_1x20_P2.54mm_Vertical -> Connector_PinHeader_2.54mm:PinHeader_1x20_P2.54mm_Vertical
- U2: footprint YAAJ_Pills:YAAJ_WeAct_BlackPill_2 -> synth:MINISTM32F4X1; now not fitted; now left out of the parts list
Connections:
- net 3V3: now also J10.20 (Pin_20), J11.3 (Pin_3)
- net C0: now also J7.16 (Pin_16); no longer J7.1 (Pin_1)
- net C1: now also J7.15 (Pin_15); no longer J7.2 (Pin_2)
- net C10: now also J7.6 (Pin_6); no longer J7.11 (Pin_11)
- net C11: now also J7.5 (Pin_5); no longer J7.12 (Pin_12)
- net C12: now also J7.4 (Pin_4); no longer J7.13 (Pin_13)
- net C13: now also J7.3 (Pin_3); no longer J7.14 (Pin_14)
- net C14: now also J7.2 (Pin_2); no longer J7.15 (Pin_15)
- net C15: now also J7.1 (Pin_1); no longer J7.16 (Pin_16)
- net C2: now also J7.14 (Pin_14); no longer J7.3 (Pin_3)
- net C3: now also J7.13 (Pin_13); no longer J7.4 (Pin_4)
- net C4: now also J7.12 (Pin_12); no longer J7.5 (Pin_5)
- net C5: now also J7.11 (Pin_11); no longer J7.6 (Pin_6)
- net C6: now also J7.10 (Pin_10); no longer J7.7 (Pin_7)
- net C7: now also J7.9 (Pin_9); no longer J7.8 (Pin_8)
- net C8: now also J7.8 (Pin_8); no longer J7.9 (Pin_9)
- net C9: now also J7.7 (Pin_7); no longer J7.10 (Pin_10)
- net D_5V: now also J10.18 (Pin_18), J11.1 (Pin_1)
- net GND: now also J10.19 (Pin_19), J11.2 (Pin_2)
- net PA0: now also J11.15 (Pin_15)
- net PA1: now also J11.14 (Pin_14)
- net PA10: now also J10.7 (Pin_7)
- net PA11: now also J10.8 (Pin_8)
- net PA12: now also J10.9 (Pin_9)
- net PA15: now also J10.10 (Pin_10)
- net PA2: now also J11.13 (Pin_13)
- net PA3: now also J11.12 (Pin_12)
- net PA4: now also J11.11 (Pin_11)
- net PA5: now also J11.10 (Pin_10)
- net PA6: now also J11.9 (Pin_9)
- net PA7: now also J11.8 (Pin_8)
- net PA8: now also J10.5 (Pin_5)
- net PA9: now also J10.6 (Pin_6)
- net PB0: now also J8.1 (Pin_1), J11.7 (Pin_7); no longer J8.5 (Pin_5)
- net PB1: now also J11.6 (Pin_6)
- net PB10: now also J11.4 (Pin_4)
- net PB12: now also J10.1 (Pin_1)
- net PB13: now also J10.2 (Pin_2)
- net PB14: now also J10.3 (Pin_3)
- net PB15: now also J8.5 (Pin_5), J10.4 (Pin_4); no longer J8.1 (Pin_1)
- net PB2: now also J11.5 (Pin_5)
- net PB3: now also J10.11 (Pin_11)
- net PB4: now also J10.12 (Pin_12)
- net PB5: now also J10.13 (Pin_13)
- net PB6: now also J10.14 (Pin_14)
- net PB7: now also J10.15 (Pin_15)
- net PB8: now also J10.16 (Pin_16)
- net PB9: now also J10.17 (Pin_17)
- net PC13: now also J11.19 (Pin_19)
- net PC14: now also J11.18 (Pin_18)
- net PC15: now also J11.17 (Pin_17)
- net RES: now also J11.16 (Pin_16)
- net VBat: now also J11.20 (Pin_20)
Other:
- moved on the sheet: J5, J6, J8, U3
