File: syth_mcu/syth_mcu.kicad_pcb (KiCad board)
At the start: 2 copper layers, 154 x 100 mm, 63 parts, among them J1 Conn_01x05, J10 Conn_01x20, J11 Conn_01x20, J2 Conn_01x05, J3 USB_C_Receptacle_PowerOnly_6P, J4 AudioPlug3, J5 Conn_01x20, J6 Conn_01x20, J7 Conn_01x16, J8 Conn_01x08, Q1 SI2307DS, Q2 SI2304DS, Q3 SI2307DS, Q4 SI2304DS, SW1 SW_Push, SW2 SW_Push, SW3 SW_Push, SW4 SW_Push, SW5 SW_Push, SW6 SW_Push, U3 AMS1117-3.3, U4 AMS1117-3.3, U5 TFT_320x240

Commit message: kicad: update pcb/sch/wrl
Parts:
- moved G*** 25.8 mm to (107.7, 139.5)
- moved H6 6.56 mm to (126.9, 113.7)
- moved H1 6.56 mm to (60.9, 113.7)
- moved H2 6.56 mm to (70.9, 113.7)
- moved H3 6.56 mm to (82.9, 113.7)
- moved H4 6.56 mm to (94.9, 113.7)
- moved H5 6.56 mm to (104.9, 113.7)
- moved H12 6.44 mm to (193.0, 113.7)
- moved H7 6.44 mm to (136.0, 113.7)
- moved RV1 5.44 mm to (71.1, 131.8)
- moved RV4 5.44 mm to (123.7, 131.8)
- moved RV2 5.44 mm to (88.6, 131.8)
- moved RV3 5.44 mm to (106.2, 131.8)
- moved RV5 5.44 mm to (141.2, 131.8)
- moved H10 4.45 mm to (171.0, 113.7)
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Connections:
- J7 pad 1: C15 -> C0
- J7 pad 10: C6 -> C9
- J7 pad 11: C5 -> C10
- J7 pad 12: C4 -> C11
- J7 pad 13: C3 -> C12
- J7 pad 14: C2 -> C13
- J7 pad 15: C1 -> C14
- J7 pad 16: C0 -> C15
- J7 pad 2: C14 -> C1
- J7 pad 3: C13 -> C2
- J7 pad 4: C12 -> C3
- J7 pad 5: C11 -> C4
- J7 pad 6: C10 -> C5
- J7 pad 7: C9 -> C6
- J7 pad 8: C8 -> C7
- J7 pad 9: C7 -> C8
- J8 pad 3: PB2 -> PA7
- J8 pad 4: PB1 -> PA6
- J8 pad 5: PB10 -> PA5
Other:
- board text added: "Made By 67011178 Napaul I. 67011246 Pavikan B. 67011214 Nuttawee W. 67011594 Chuthathip T. 67011220 Pacharapol P. 67011671 Tithipan T."
- board text removed: "Made By 67011178 Napaul I. 67011214 Nuttawee W. 67011220 Pacharapol P. 67011246 Pavikan B. 67011594 Chuthathip T. 67011671 Tithipan T."
