File: syth_mcu/MuxAnalog.kicad_sch (KiCad schematic)
At the start: 24 parts

Commit message: v2 schematic merge, power and signal routing
Parts:
- H1, H10, H11, H12, H2, H3, H4, H5, H6, H7, H8, H9: footprint Package_TO_SOT_THT:TO-92_Inline -> synth:TO-92_Inline_AH3503
Changed lines of the file:
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@@
 	(global_label "AMS2_3.3V"
 		(shape input)
-		(at 0.0794 1.3498 0)
-		(fields_autoplaced yes)
-		(effects
-			(font
-				(size 1.27 1.27)
-			)
-			(justify left)
-		)
-		(property "Intersheetrefs" "${INTERSHEET_REFS}"
-			(at 13.1036 1.3498 0)
-			(hide yes)
-			(show_name no)
-			(do_not_autoplace no)
-			(effects
-				(font
-					(size 1.27 1.27)
-				)
-				(justify left)
-			)
-		)
-	)
-	(global_label "AMS2_3.3V"
-		(shape input)
 		(at 71.12 90.17 270)
 		(fields_autoplaced yes)
@@
 			)
 		)
-		(property "Footprint" "Package_TO_SOT_THT:TO-92_Inline"
+		(property "Footprint" "synth:TO-92_Inline_AH3503"
 			(at 109.22 29.21 0)
 			(hide yes)
@@
 			)
 		)
-		(property "Footprint" "Package_TO_SOT_THT:TO-92_Inline"
+		(property "Footprint" "synth:TO-92_Inline_AH3503"
 			(at 73.66 29.21 0)
 			(hide yes)
@@
 			)
 		)
-		(property "Footprint" "Package_TO_SOT_THT:TO-92_Inline"
+		(property "Footprint" "synth:TO-92_Inline_AH3503"
 			(at 118.11 29.21 0)
 			(hide yes)
@@
 			)
 		)
-		(property "Footprint" "Package_TO_SOT_THT:TO-92_Inline"
+		(property "Footprint" "synth:TO-92_Inline_AH3503"
 			(at 100.33 29.21 0)
 			(hide yes)
@@
 			)
 		)
-		(property "Footprint" "Package_TO_SOT_THT:TO-92_Inline"
+		(property "Footprint" "synth:TO-92_Inline_AH3503"
 			(at 127 29.21 0)
 			(hide yes)
@@
 			)
 		)
-		(property "Footprint" "Package_TO_SOT_THT:TO-92_Inline"
+		(property "Footprint" "synth:TO-92_Inline_AH3503"
 			(at 144.78 29.21 0)
 			(hide yes)
@@
 			)
 		)
-		(property "Footprint" "Package_TO_SOT_THT:TO-92_Inline"
+		(property "Footprint" "synth:TO-92_Inline_AH3503"
 			(at 46.99 29.21 0)
 			(hide yes)
@@
 			)
 		)
-		(property "Footprint" "Package_TO_SOT_THT:TO-92_Inline"
+		(property "Footprint" "synth:TO-92_Inline_AH3503"
 			(at 82.55 29.21 0)
 			(hide yes)
@@
 			)
 		)
-		(property "Footprint" "Package_TO_SOT_THT:TO-92_Inline"
+		(property "Footprint" "synth:TO-92_Inline_AH3503"
 			(at 91.44 29.21 0)
 			(hide yes)
@@
 			)
 		)
-		(property "Footprint" "Package_TO_SOT_THT:TO-92_Inline"
+		(property "Footprint" "synth:TO-92_Inline_AH3503"
 			(at 135.89 29.21 0)
 			(hide yes)
@@
 			)
 		)
-		(property "Footprint" "Package_TO_SOT_THT:TO-92_Inline"
+		(property "Footprint" "synth:TO-92_Inline_AH3503"
 			(at 64.77 29.21 0)
 			(hide yes)
@@
 			)
 		)
-		(property "Footprint" "Package_TO_SOT_THT:TO-92_Inline"
+		(property "Footprint" "synth:TO-92_Inline_AH3503"
 			(at 55.88 29.21 0)
 			(hide yes)
