File: syth_mcu/_restore_backup_2026-09-01T22-17-18-245/dac-pchannel.kicad_sch (KiCad schematic)
At the start: 23 parts, among them J4 AudioPlug3, Q1 SI2307DS, Q2 SI2304DS, Q3 SI2307DS, Q4 SI2304DS

Commit message: synth: fix 3D models, source real jack part, rename syth big -> syth_mcu
3D model fixes (all footprints were pointing at broken/missing paths):
- Pot (RV1-7): Alps RK09K STEP wired via project-relative ${KIPRJMOD} path
- Pogo connector (J1/J2): real magnetic pogo STEP, replaced broken
  pogo5.3dshapes reference that pointed at a folder that never existed
- Switch (SW1-6): sourced Kailh LP Choc STEP + MX-Alps-Choc-1U hybrid
  footprint (drop-in candidate for existing Cherry MX pad pattern)
- Jack (J4): sourced real, cheap (~35 THB), Thailand-buyable PJ-316 part
  via easyeda2kicad (LCSC C2884936) - symbol, footprint, and 3D model
  all pulled fresh

All models now use ${KIPRJMOD}-relative paths under syth_mcu/local_3dmodels/
so they resolve on any machine after git pull, not just this one.

Also folds in the syth big -> syth_mcu folder rename and other pending
schematic/production file changes.
Parts:
- C1, C2: value 80nF -> 100nF; footprint Capacitor_THT:CP_Radial_D4.0mm_P2.00mm -> Capacitor_THT:C_Disc_D5.0mm_W2.5mm_P2.50mm
- C6, C8: footprint Capacitor_THT:CP_Radial_D4.0mm_P2.00mm -> Capacitor_THT:CP_Radial_D5.0mm_P2.00mm
- J4: footprint synth:CONN-TH_PJ-316 -> Connector_Audio:Jack_3.5mm_CUI_SJ1-3533NG_Horizontal
- RV6, RV7: footprint synth:Potentiometer_Alps_RK09K_Single_Vertical -> Potentiometer_THT:Potentiometer_Bourns_3296W_Vertical
Changed lines of the file:
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@@
 			)
 		)
-		(property "Footprint" "synth:CONN-TH_PJ-316"
+		(property "Footprint" "Connector_Audio:Jack_3.5mm_CUI_SJ1-3533NG_Horizontal"
 			(at 58.42 153.67 0)
 			(hide yes)
@@
 			)
 		)
-		(property "Footprint" "synth:Potentiometer_Alps_RK09K_Single_Vertical"
+		(property "Footprint" "Potentiometer_THT:Potentiometer_Bourns_3296W_Vertical"
 			(at 104.14 72.39 0)
 			(hide yes)
@@
 		)
 		(property "Description" "Potentiometer"
-			(at 104.14 72.39 0)
-			(hide yes)
-			(show_name no)
-			(do_not_autoplace no)
-			(effects
-				(font
-					(size 1.27 1.27)
-				)
-			)
-		)
-		(property "Sim.Device" "R"
-			(at 104.14 72.39 0)
-			(hide yes)
-			(show_name no)
-			(do_not_autoplace no)
-			(effects
-				(font
-					(size 1.27 1.27)
-				)
-			)
-		)
-		(property "Sim.Type" "POT"
-			(at 104.14 72.39 0)
-			(hide yes)
-			(show_name no)
-			(do_not_autoplace no)
-			(effects
-				(font
-					(size 1.27 1.27)
-				)
-			)
-		)
-		(property "Sim.Pins" "1=r0 2=wiper 3=r1"
 			(at 104.14 72.39 0)
 			(hide yes)
@@
 			)
 		)
-		(property "Value" "80nF"
+		(property "Value" "100nF"
 			(at 77.47 67.3099 0)
 			(show_name no)
@@
 			)
 		)
-		(property "Footprint" "Capacitor_THT:CP_Radial_D4.0mm_P2.00mm"
+		(property "Footprint" "Capacitor_THT:C_Disc_D5.0mm_W2.5mm_P2.50mm"
 			(at 80.3148 69.85 0)
 			(hide yes)
@@
 			)
 		)
-		(property "Footprint" "synth:Potentiometer_Alps_RK09K_Single_Vertical"
+		(property "Footprint" "Potentiometer_THT:Potentiometer_Bourns_3296W_Vertical"
 			(at 104.14 127 0)
 			(hide yes)
@@
 		)
 		(property "Description" "Potentiometer"
-			(at 104.14 127 0)
-			(hide yes)
-			(show_name no)
-			(do_not_autoplace no)
-			(effects
-				(font
-					(size 1.27 1.27)
-				)
-			)
-		)
-		(property "Sim.Device" "R"
-			(at 104.14 127 0)
-			(hide yes)
-			(show_name no)
-			(do_not_autoplace no)
-			(effects
-				(font
-					(size 1.27 1.27)
-				)
-			)
-		)
-		(property "Sim.Type" "POT"
-			(at 104.14 127 0)
-			(hide yes)
-			(show_name no)
-			(do_not_autoplace no)
-			(effects
-				(font
-					(size 1.27 1.27)
-				)
-			)
-		)
-		(property "Sim.Pins" "1=r0 2=wiper 3=r1"
 			(at 104.14 127 0)
 			(hide yes)
@@
 			)
 		)
-		(property "Value" "80nF"
+		(property "Value" "100nF"
 			(at 77.47 121.9199 0)
 			(show_name no)
@@
 			)
 		)
-		(property "Footprint" "Capacitor_THT:CP_Radial_D4.0mm_P2.00mm"
+		(property "Footprint" "Capacitor_THT:C_Disc_D5.0mm_W2.5mm_P2.50mm"
 			(at 80.3148 124.46 0)
 			(hide yes)
@@
 			)
 		)
-		(property "Footprint" "Capacitor_THT:CP_Radial_D4.0mm_P2.00mm"
+		(property "Footprint" "Capacitor_THT:CP_Radial_D5.0mm_P2.00mm"
 			(at 103.1748 120.65 0)
 			(hide yes)
@@
 			)
 		)
-		(property "Footprint" "Capacitor_THT:CP_Radial_D4.0mm_P2.00mm"
+		(property "Footprint" "Capacitor_THT:CP_Radial_D5.0mm_P2.00mm"
 			(at 103.1748 66.04 0)
 			(hide yes)
