File: syth_mcu/_restore_backup_2026-09-01T22-17-18-245/syth_mcu.kicad_sch (KiCad schematic)
At the start: 40 parts, among them J1 Conn_01x05, J10 Conn_01x20, J11 Conn_01x20, J2 Conn_01x05, J3 USB_C_Receptacle_PowerOnly_6P, J5 Conn_01x20, J6 Conn_01x20, J7 Conn_01x16, J8 Conn_01x08, SW1 SW_Push, SW2 SW_Push, SW3 SW_Push, SW4 SW_Push, SW5 SW_Push, SW6 SW_Push, U2 YAAJ_WeAct_BlackPill_Part_Like, U3 AMS1117-3.3, U4 AMS1117-3.3, U5 TFT_320x240

Commit message: synth: fix 3D models, source real jack part, rename syth big -> syth_mcu
3D model fixes (all footprints were pointing at broken/missing paths):
- Pot (RV1-7): Alps RK09K STEP wired via project-relative ${KIPRJMOD} path
- Pogo connector (J1/J2): real magnetic pogo STEP, replaced broken
  pogo5.3dshapes reference that pointed at a folder that never existed
- Switch (SW1-6): sourced Kailh LP Choc STEP + MX-Alps-Choc-1U hybrid
  footprint (drop-in candidate for existing Cherry MX pad pattern)
- Jack (J4): sourced real, cheap (~35 THB), Thailand-buyable PJ-316 part
  via easyeda2kicad (LCSC C2884936) - symbol, footprint, and 3D model
  all pulled fresh

All models now use ${KIPRJMOD}-relative paths under syth_mcu/local_3dmodels/
so they resolve on any machine after git pull, not just this one.

Also folds in the syth big -> syth_mcu folder rename and other pending
schematic/production file changes.
Parts:
- removed C9: C_Small, Capacitor_THT:C_Disc_D5.0mm_W2.5mm_P2.50mm, symbol Device:C_Small
- removed H1, H2, H3, H4, H5: (no value), Package_TO_SOT_THT:TO-92_Inline, symbol synth:H3503
- removed SW6: SW_Push, synth:MX-Alps-Choc-1U, symbol Switch:SW_Push
- added J9: Conn_01x07, Connector_PinSocket_2.54mm:PinSocket_1x07_P2.54mm_Vertical, symbol Connector_Generic:Conn_01x07
- D1: value SS34 -> SS14
- RV1, RV2, RV3, RV4, RV5: footprint synth:Potentiometer_Alps_RK09K_Single_Vertical -> Potentiometer_THT:Potentiometer_Alps_RK09K_Single_Vertical
- SW1, SW2, SW3, SW4, SW5: footprint synth:MX-Alps-Choc-1U -> Button_Switch_Keyboard:SW_Cherry_MX_1.00u_PCB
- U2: footprint Kicad-STM32:YAAJ_WeAct_BlackPill2 -> synth:MINISTM32F4X1
- U5: footprint Connector_PinHeader_2.54mm:PinHeader_1x14_P2.54mm_Vertical -> Connector_PinSocket_2.54mm:PinSocket_1x14_P2.54mm_Vertical
Connections:
- net AMS1_3.3V: now also H10.2 (GND), H11.2 (GND), H12.2 (GND), H9.2 (GND), J9.6 (Pin_6); no longer H10.1 (VCC), H11.1 (VCC), H12.1 (VCC), H9.1 (VCC)
- net C0: now also J9.1 (Pin_1)
- net C1: now also J9.2 (Pin_2)
- net C2: now also J9.3 (Pin_3)
- net C3: now also J9.4 (Pin_4)
- net C4: now also J9.5 (Pin_5)
- net GND: now also H10.1 (VCC), H11.1 (VCC), H12.1 (VCC), H9.1 (VCC), J9.7 (Pin_7); no longer H10.2 (GND), H11.2 (GND), H12.2 (GND), H9.2 (GND), J1.5 (Pin_5), J2.5 (Pin_5)
- net PA11: now also J2.5 (Pin_5)
- net PA12: now also J1.5 (Pin_5)
- net PA5: now also U5.7 (SCK)
- net PA7: now also U5.6 (MOSI)
- net PB0: now also J8.1 (Pin_1); no longer J8.2 (Pin_2)
- net PB1: no longer J8.4 (Pin_4)
- net PB10: no longer J8.5 (Pin_5)
- net PB12: now also SW5.2; no longer SW1.2
- net PB13: now also J8.3 (Pin_3); no longer U5.7 (SCK)
- net PB14: now also J8.2 (Pin_2); no longer U5.6 (MOSI)
- net PB15: now also J8.5 (Pin_5); no longer SW2.2
- net PB2: now also J8.4 (Pin_4); no longer J8.3 (Pin_3)
- net PB4: now also SW1.2; no longer SW3.2
- net PB5: now also SW2.2; no longer J8.1 (Pin_1), SW4.2
- net PB8: now also SW3.2; no longer SW5.2
- net PB9: now also SW4.2
- no-connect marks 36 -> 7
Other:
- note removed: "ENN"
- moved on the sheet: D1, J1, J10, J11, J2, J3, J5, J6, J7, J8, R1, R2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
