File: syth_mcu/_restore_backup_2026-09-01T22-17-18-245/untitled.kicad_sch (KiCad schematic)
At the start: 6 parts, among them J10 Conn_01x07

Commit message: synth: fix 3D models, source real jack part, rename syth big -> syth_mcu
3D model fixes (all footprints were pointing at broken/missing paths):
- Pot (RV1-7): Alps RK09K STEP wired via project-relative ${KIPRJMOD} path
- Pogo connector (J1/J2): real magnetic pogo STEP, replaced broken
  pogo5.3dshapes reference that pointed at a folder that never existed
- Switch (SW1-6): sourced Kailh LP Choc STEP + MX-Alps-Choc-1U hybrid
  footprint (drop-in candidate for existing Cherry MX pad pattern)
- Jack (J4): sourced real, cheap (~35 THB), Thailand-buyable PJ-316 part
  via easyeda2kicad (LCSC C2884936) - symbol, footprint, and 3D model
  all pulled fresh

All models now use ${KIPRJMOD}-relative paths under syth_mcu/local_3dmodels/
so they resolve on any machine after git pull, not just this one.

Also folds in the syth big -> syth_mcu folder rename and other pending
schematic/production file changes.
Parts:
- renumbered H1 to H13, H2 to H14, H3 to H15, H4 to H16, H5 to H17
Changed lines of the file:
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@@
 		(dnp no)
 		(fields_autoplaced yes)
-		(property "Reference" "H3"
-			(at 138.43 36.83 90)
-			(show_name no)
-			(do_not_autoplace no)
-			(effects
-				(font
-					(size 1.27 1.27)
-				)
+		(property "Reference" "H15"
+			(at 138.4299 38.1 0)
+			(show_name no)
+			(do_not_autoplace no)
+			(effects
+				(font
+					(size 1.27 1.27)
+				)
+				(justify left)
 			)
 		)
@@
 			(project "syth_mcu"
 				(path "/b9b81bb9-b7d6-4262-8e2b-de009d5ce128"
-					(reference "H3")
+					(reference "H15")
 					(unit 1)
 				)
@@
 		(dnp no)
 		(fields_autoplaced yes)
-		(property "Reference" "H2"
-			(at 129.54 36.83 90)
-			(show_name no)
-			(do_not_autoplace no)
-			(effects
-				(font
-					(size 1.27 1.27)
-				)
+		(property "Reference" "H14"
+			(at 129.5399 38.1 0)
+			(show_name no)
+			(do_not_autoplace no)
+			(effects
+				(font
+					(size 1.27 1.27)
+				)
+				(justify left)
 			)
 		)
@@
 			(project "syth_mcu"
 				(path "/b9b81bb9-b7d6-4262-8e2b-de009d5ce128"
-					(reference "H2")
+					(reference "H14")
 					(unit 1)
 				)
@@
 		(dnp no)
 		(fields_autoplaced yes)
-		(property "Reference" "H5"
-			(at 161.29 42.5449 90)
-			(show_name no)
-			(do_not_autoplace no)
-			(effects
-				(font
-					(size 1.27 1.27)
-				)
-				(justify right)
+		(property "Reference" "H17"
+			(at 156.2099 38.1 0)
+			(show_name no)
+			(do_not_autoplace no)
+			(effects
+				(font
+					(size 1.27 1.27)
+				)
+				(justify left)
 			)
 		)
@@
 			(project "syth_mcu"
 				(path "/b9b81bb9-b7d6-4262-8e2b-de009d5ce128"
-					(reference "H5")
+					(reference "H17")
 					(unit 1)
 				)
@@
 		(in_pos_files yes)
 		(dnp no)
-		(fields_autoplaced yes)
 		(property "Reference" "J10"
-			(at 118.11 71.1199 0)
-			(show_name no)
-			(do_not_autoplace no)
-			(effects
-				(font
-					(size 1.27 1.27)
-				)
-				(justify left)
+			(at 120.65 86.36 0)
+			(show_name no)
+			(do_not_autoplace no)
+			(effects
+				(font
+					(size 1.27 1.27)
+				)
 			)
 		)
 		(property "Value" "Conn_01x07"
-			(at 118.11 73.6599 0)
-			(show_name no)
-			(do_not_autoplace no)
-			(effects
-				(font
-					(size 1.27 1.27)
-				)
-				(justify left)
+			(at 120.65 83.82 0)
+			(show_name no)
+			(do_not_autoplace no)
+			(effects
+				(font
+					(size 1.27 1.27)
+				)
 			)
 		)
@@
 		(dnp no)
 		(fields_autoplaced yes)
-		(property "Reference" "H1"
-			(at 120.65 36.83 90)
-			(show_name no)
-			(do_not_autoplace no)
-			(effects
-				(font
-					(size 1.27 1.27)
-				)
+		(property "Reference" "H13"
+			(at 120.6499 38.1 0)
+			(show_name no)
+			(do_not_autoplace no)
+			(effects
+				(font
+					(size 1.27 1.27)
+				)
+				(justify left)
 			)
 		)
@@
 			(project "syth_mcu"
 				(path "/b9b81bb9-b7d6-4262-8e2b-de009d5ce128"
-					(reference "H1")
+					(reference "H13")
 					(unit 1)
 				)
@@
 		)
 		(property "Value" "GND"
-			(at 127 83.82 90)
-			(show_name no)
-			(do_not_autoplace no)
-			(effects
-				(font
-					(size 1.27 1.27)
-				)
+			(at 129.54 80.0099 90)
+			(show_name no)
+			(do_not_autoplace no)
+			(effects
+				(font
+					(size 1.27 1.27)
+				)
+				(justify right)
 			)
 		)
@@
 		(dnp no)
 		(fields_autoplaced yes)
-		(property "Reference" "H4"
-			(at 147.32 36.83 90)
-			(show_name no)
-			(do_not_autoplace no)
-			(effects
-				(font
-					(size 1.27 1.27)
-				)
+		(property "Reference" "H16"
+			(at 147.3199 38.1 0)
+			(show_name no)
+			(do_not_autoplace no)
+			(effects
+				(font
+					(size 1.27 1.27)
+				)
+				(justify left)
 			)
 		)
@@
 			(project "syth_mcu"
 				(path "/b9b81bb9-b7d6-4262-8e2b-de009d5ce128"
-					(reference "H4")
-					(unit 1)
-				)
+					(reference "H16")
+					(unit 1)
+				)
